File: electronics/KeyModule/KeyModule.kicad_sch (KiCad schematic)
At the start: 13 parts, among them SW1 SW_Push, SW2 SW_Push, SW3 SW_Push, SW4 SW_Push, SW5 SW_Push, U1 74HC165

Commit message: Split module connectors into three 1x3 pairs and add the pin bend jig
Schematic: J_LEFT1 and J_RIGHT1 (1x9) become J_LEFT1..3 sockets and
J_RIGHT1..3 headers with the Harwin footprints assigned, pins kept on
the same sheet positions so the wiring is unchanged; ERC clean.
Electronics.md documents the per-connector pinout. roamy-v3.py grows a
two-part jig that bends the header pins to the joint angle before
soldering. The joint drawing is embedded in both design docs.

Co-Authored-By: Claude Fable 5.1 <noreply@anthropic.com>
Parts:
- removed J_LEFT1: Conn_01x09, Connector_PinHeader_2.54mm:PinHeader_1x09_P2.54mm_Vertical_SMD_Pin1Right, symbol Connector_Generic:Conn_01x09
- removed J_RIGHT1: Conn_01x09, Connector_PinHeader_2.54mm:PinHeader_1x09_P2.54mm_Vertical_SMD_Pin1Left, symbol Connector_Generic:Conn_01x09
- added J_LEFT1, J_LEFT2, J_LEFT3: M20-7910342R, Library:Harwin_M20-791_1x03_Horizontal_SMD, symbol Connector_Generic:Conn_01x03
- added J_RIGHT1, J_RIGHT2, J_RIGHT3: M20-8890345R, Library:Harwin_M20-889_1x03_Horizontal_SMD, symbol Connector_Generic:Conn_01x03
Connections:
- net +3.3V: now also J_LEFT1.2 (Pin_2), J_RIGHT1.2 (Pin_2)
- net +5V: now also J_LEFT1.1 (Pin_1), J_RIGHT1.1 (Pin_1)
- net CLK: now also J_LEFT2.1 (Pin_1), J_RIGHT2.1 (Pin_1)
- net DATA_IN: now also J_LEFT2.2 (Pin_2)
- net DATA_OUT: now also J_RIGHT2.2 (Pin_2)
- net GND: now also J_LEFT1.3 (Pin_3), J_RIGHT1.3 (Pin_3)
- net LED: now also J_LEFT3.1 (Pin_1), J_RIGHT3.1 (Pin_1)
- net PL: now also J_LEFT2.3 (Pin_3), J_RIGHT2.3 (Pin_3)
- net SCL: now also J_LEFT3.3 (Pin_3), J_RIGHT3.3 (Pin_3)
- net SDA: now also J_LEFT3.2 (Pin_2), J_RIGHT3.2 (Pin_2)

Commit message: Route the key module
All copper on the back except five 0805 pull-downs, which move to the
front between switches where nothing else lives. Row 2 of the
interconnect becomes CLK / PL / DATA: DATA on the bottom pin is the
only pin whose track can leave the pad without crossing a pass-through.
Choc hotswap sockets, their pads and outline move to the back of the
switch footprint, where the socket physically mounts. GND is the zone
on both layers, stitched by five vias. kicad-cli DRC with schematic
parity: no violations, no unconnected items.

Co-Authored-By: Claude Fable 5.1 <noreply@anthropic.com>
Connections:
- net DATA_IN: now also J_LEFT2.3 (Pin_3); no longer J_LEFT2.2 (Pin_2)
- net DATA_OUT: now also J_RIGHT2.3 (Pin_3); no longer J_RIGHT2.2 (Pin_2)
- net PL: now also J_LEFT2.2 (Pin_2), J_RIGHT2.2 (Pin_2); no longer J_LEFT2.3 (Pin_3), J_RIGHT2.3 (Pin_3)
Changed lines of the file:
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@@
 		)
 	)
-	(label "DATA_IN"
+	(label "PL"
 		(at 53.34 85.09 0)
 		(effects
@@
 		)
 	)
-	(label "PL"
+	(label "DATA_IN"
 		(at 53.34 87.63 0)
 		(effects
@@
 		)
 	)
-	(label "DATA_OUT"
+	(label "PL"
 		(at 144.78 85.09 180)
 		(effects
@@
 		)
 	)
-	(label "PL"
+	(label "DATA_OUT"
 		(at 144.78 87.63 180)
 		(effects
