File: electronics/KeyModule/KeyModule.kicad_sch (KiCad schematic)
At the start: 17 parts, among them SW1 SW_Push, SW2 SW_Push, SW3 SW_Push, SW4 SW_Push, SW5 SW_Push, U1 74HC165

Commit message: Add 100 nF decoupling for the 165 and export fab files
Electronics.md promised decoupling and the schematic had none. C1 sits
on the front beside U1, fed from the +3.3V branch. ERC clean, DRC with
parity clean. fab/KeyModule-gerbers.zip holds gerbers and drills for
this revision.

Co-Authored-By: Claude Fable 5.1 <noreply@anthropic.com>
Parts:
- added C1: 100nF, Capacitor_SMD:C_0805_2012Metric, symbol Device:C
Connections:
- net +3.3V: now also C1.1
- net GND: now also C1.2

Commit message: Part numbers on every symbol and a BOM for ordering
LCSC numbers for the 165, resistors, cap, sockets and the Harwin
receptacle; the Harwin header is DigiKey only. fab/KeyModule-bom.csv is
the kicad-cli export plus the hotswap sockets, which live inside the
switch footprint and have no symbol of their own.

Co-Authored-By: Claude Fable 5.1 <noreply@anthropic.com>
Parts:
- C1: Ideal Part Number (none) -> CC0805KRX7R9BB104; LCSC Part # (none) -> C49678; Order Link (none) -> https://www.lcsc.com/product-detail/C49678.html; Vendor (none) -> LCSC
- J_LEFT1, J_LEFT2, J_LEFT3: LCSC Part # (none) -> C3321821; Order Link https://www.digikey.se/en/products/detail/harwin-inc/M20-79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 -> https://jlcpcb.com/partdetail/Harwin-M207910342R/C3321821; Vendor Harwin -> LCSC
- J_RIGHT1, J_RIGHT2, J_RIGHT3: Order Link https://www.harwin.com/products/M20-8890345R -> https://www.digikey.com/en/products/detail/harwin-inc/M20-8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; Vendor Harwin -> DigiKey
- R1, R2, R3, R4, R5: Ideal Part Number (none) -> 0805W8F1002T5E; LCSC Part # (none) -> C17414; Order Link (none) -> https://www.lcsc.com/product-detail/C17414.html; Vendor (none) -> LCSC
- U1: LCSC Part # (none) -> C5613; Order Link https://www.digikey.se/sv/products/detail/nexperia-usa-inc/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 -> https://www.lcsc.com/product-detail/C5613.html; Vendor Nexperia USA Inc. -> LCSC
Changed lines of the file:
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@@
 			)
 		)
-		(property "Order Link" "https://www.digikey.se/sv/products/detail/nexperia-usa-inc/74HC165D-653/763013"
+		(property "Order Link" "https://www.lcsc.com/product-detail/C5613.html"
 			(at 118.11 80.01 0)
 			(hide yes)
@@
 			)
 		)
-		(property "Vendor" "Nexperia USA Inc."
+		(property "Vendor" "LCSC"
+			(at 118.11 80.01 0)
+			(hide yes)
+			(show_name no)
+			(do_not_autoplace no)
+			(effects
+				(font
+					(size 1.27 1.27)
+				)
+			)
+		)
+		(property "LCSC Part #" "C5613"
 			(at 118.11 80.01 0)
 			(hide yes)
@@
 			)
 		)
-		(property "Ideal Part Number" ""
+		(property "Ideal Part Number" "0805W8F1002T5E"
 			(at 88.9 111.76 90)
 			(hide yes)
@@
 			)
 		)
-		(property "Order Link" ""
+		(property "Order Link" "https://www.lcsc.com/product-detail/C17414.html"
 			(at 88.9 111.76 90)
 			(hide yes)
@@
 			)
 		)
-		(property "Vendor" ""
+		(property "Vendor" "LCSC"
 			(at 88.9 111.76 90)
 			(hide yes)
@@
 			)
 		)
+		(property "LCSC Part #" "C17414"
+			(at 88.9 111.76 0)
+			(hide yes)
+			(show_name no)
+			(do_not_autoplace no)
+			(effects
+				(font
+					(size 1.27 1.27)
+				)
+			)
+		)
 		(pin "1"
 		)
@@
 			)
 		)
-		(property "Order Link" "https://www.digikey.se/en/products/detail/harwin-inc/M20-7910342R/6559281"
+		(property "Order Link" "https://jlcpcb.com/partdetail/Harwin-M207910342R/C3321821"
+			(at 48.26 85.09 0)
+			(hide yes)
+			(show_name no)
+			(do_not_autoplace no)
+			(effects
+				(font
+					(size 1.27 1.27)
+				)
+			)
+		)
+		(property "Vendor" "LCSC"
 			(at 48.26 85.09 0)
 			(hide yes)
@@
 			)
 		)
-		(property "Vendor" "Harwin"
+		(property "LCSC Part #" "C3321821"
 			(at 48.26 85.09 0)
 			(hide yes)
@@
 			)
 		)
-		(property "Ideal Part Number" ""
+		(property "Ideal Part Number" "0805W8F1002T5E"
 			(at 88.9 83.82 90)
 			(hide yes)
@@
 			)
 		)
-		(property "Order Link" ""
+		(property "Order Link" "https://www.lcsc.com/product-detail/C17414.html"
 			(at 88.9 83.82 90)
 			(hide yes)
@@
 			)
 		)
-		(property "Vendor" ""
+		(property "Vendor" "LCSC"
 			(at 88.9 83.82 90)
 			(hide yes)
@@
 			)
 		)
+		(property "LCSC Part #" "C17414"
+			(at 88.9 83.82 0)
+			(hide yes)
+			(show_name no)
+			(do_not_autoplace no)
+			(effects
+				(font
+					(size 1.27 1.27)
+				)
+			)
+		)
 		(pin "2"
 		)
@@
 			)
 		)
-		(property "Ideal Part Number" ""
+		(property "Ideal Part Number" "0805W8F1002T5E"
 			(at 88.9 127 90)
 			(hide yes)
@@
 			)
 		)
-		(property "Order Link" ""
+		(property "Order Link" "https://www.lcsc.com/product-detail/C17414.html"
 			(at 88.9 127 90)
 			(hide yes)
@@
 			)
 		)
-		(property "Vendor" ""
+		(property "Vendor" "LCSC"
 			(at 88.9 127 90)
 			(hide yes)
@@
 			)
 		)
+		(property "LCSC Part #" "C17414"
+			(at 88.9 127 0)
+			(hide yes)
+			(show_name no)
+			(do_not_autoplace no)
+			(effects
+				(font
+					(size 1.27 1.27)
+				)
+			)
+		)
 		(pin "1"
 		)
@@
 			)
 		)
-		(property "Order Link" "https://www.harwin.com/products/M20-8890345R"
+		(property "Order Link" "https://www.digikey.com/en/products/detail/harwin-inc/M20-8890345R/6565723"
+			(at 149.86 92.71 0)
+			(hide yes)
+			(show_name no)
+			(do_not_autoplace no)
+			(effects
+				(font
+					(size 1.27 1.27)
+				)
+			)
+		)
+		(property "Vendor" "DigiKey"
 			(at 149.86 92.71 0)
 			(hide yes)
@@
 			)
 		)
-		(property "Vendor" "Harwin"
+		(property "LCSC Part #" ""
 			(at 149.86 92.71 0)
 			(hide yes)
@@
 			)
 		)
-		(property "Ideal Part Number" ""
+		(property "Ideal Part Number" "0805W8F1002T5E"
 			(at 88.9 97.79 90)
 			(hide yes)
@@
 			)
 		)
-		(property "Order Link" ""
+		(property "Order Link" "https://www.lcsc.com/product-detail/C17414.html"
 			(at 88.9 97.79 90)
 			(hide yes)
@@
 			)
 		)
-		(property "Vendor" ""
+		(property "Vendor" "LCSC"
 			(at 88.9 97.79 90)
 			(hide yes)
@@
 			)
 		)
+		(property "LCSC Part #" "C17414"
+			(at 88.9 97.79 0)
+			(hide yes)
+			(show_name no)
+			(do_not_autoplace no)
+			(effects
+				(font
+					(size 1.27 1.27)
+				)
+			)
+		)
 		(pin "2"
 		)
@@
 			)
 		)
-		(property "Order Link" "https://www.harwin.com/products/M20-8890345R"
+		(property "Order Link" "https://www.digikey.com/en/products/detail/harwin-inc/M20-8890345R/6565723"
 			(at 149.86 85.09 0)
 			(hide yes)
@@
 			)
 		)
-		(property "Vendor" "Harwin"
+		(property "Vendor" "DigiKey"
+			(at 149.86 85.09 0)
+			(hide yes)
+			(show_name no)
+			(do_not_autoplace no)
+			(effects
+				(font
+					(size 1.27 1.27)
+				)
+			)
+		)
+		(property "LCSC Part #" ""
 			(at 149.86 85.09 0)
 			(hide yes)
@@
 			)
 		)
-		(property "Order Link" "https://www.harwin.com/products/M20-8890345R"
+		(property "Order Link" "https://www.digikey.com/en/products/detail/harwin-inc/M20-8890345R/6565723"
 			(at 149.86 77.47 0)
 			(hide yes)
@@
 			)
 		)
-		(property "Vendor" "Harwin"
+		(property "Vendor" "DigiKey"
+			(at 149.86 77.47 0)
+			(hide yes)
+			(show_name no)
+			(do_not_autoplace no)
+			(effects
+				(font
+					(size 1.27 1.27)
+				)
+			)
+		)
+		(property "LCSC Part #" ""
 			(at 149.86 77.47 0)
 			(hide yes)
@@
 			)
 		)
-		(property "Order Link" "https://www.digikey.se/en/products/detail/harwin-inc/M20-7910342R/6559281"
+		(property "Order Link" "https://jlcpcb.com/partdetail/Harwin-M207910342R/C3321821"
+			(at 48.26 77.47 0)
+			(hide yes)
+			(show_name no)
+			(do_not_autoplace no)
+			(effects
+				(font
+					(size 1.27 1.27)
+				)
+			)
+		)
+		(property "Vendor" "LCSC"
 			(at 48.26 77.47 0)
 			(hide yes)
@@
 			)
 		)
-		(property "Vendor" "Harwin"
+		(property "LCSC Part #" "C3321821"
 			(at 48.26 77.47 0)
 			(hide yes)
@@
 			)
 		)
-		(property "Ideal Part Number" ""
+		(property "Ideal Part Number" "0805W8F1002T5E"
 			(at 88.9 69.85 90)
 			(hide yes)
@@
 			)
 		)
-		(property "Order Link" ""
+		(property "Order Link" "https://www.lcsc.com/product-detail/C17414.html"
 			(at 88.9 69.85 90)
 			(hide yes)
@@
 			)
 		)
-		(property "Vendor" ""
+		(property "Vendor" "LCSC"
 			(at 88.9 69.85 90)
 			(hide yes)
@@
 			)
 		)
+		(property "LCSC Part #" "C17414"
+			(at 88.9 69.85 0)
+			(hide yes)
+			(show_name no)
+			(do_not_autoplace no)
+			(effects
+				(font
+					(size 1.27 1.27)
+				)
+			)
+		)
 		(pin "1"
 		)
@@
 			)
 		)
-		(property "Order Link" "https://www.digikey.se/en/products/detail/harwin-inc/M20-7910342R/6559281"
+		(property "Order Link" "https://jlcpcb.com/partdetail/Harwin-M207910342R/C3321821"
 			(at 48.26 92.71 0)
 			(hide yes)
@@
 			)
 		)
-		(property "Vendor" "Harwin"
+		(property "Vendor" "LCSC"
+			(at 48.26 92.71 0)
+			(hide yes)
+			(show_name no)
+			(do_not_autoplace no)
+			(effects
+				(font
+					(size 1.27 1.27)
+				)
+			)
+		)
+		(property "LCSC Part #" "C3321821"
 			(at 48.26 92.71 0)
 			(hide yes)
@@
 			)
 		)
-		(property "Ideal Part Number" ""
+		(property "Ideal Part Number" "CC0805KRX7R9BB104"
 			(at 165.1 100.33 0)
 			(hide yes)
@@
 			)
 		)
-		(property "Order Link" ""
+		(property "Order Link" "https://www.lcsc.com/product-detail/C49678.html"
 			(at 165.1 100.33 0)
 			(hide yes)
@@
 			)
 		)
-		(property "Vendor" ""
+		(property "Vendor" "LCSC"
+			(at 165.1 100.33 0)
+			(hide yes)
+			(show_name no)
+			(do_not_autoplace no)
+			(effects
+				(font
+					(size 1.27 1.27)
+				)
+			)
+		)
+		(property "LCSC Part #" "C49678"
 			(at 165.1 100.33 0)
 			(hide yes)

Commit message: Switch the interconnect to hanxia HX PM2.54/PZ2.54 horizontal headers
Same 8.5 x 2.5 mm socket body, 2.5 mm header body, 0.64 mm square
6 mm pins and 1.25 mm pin axis as the Harwin M20 pair, and their
recommended pads land inside the existing footprints, so the board is
unchanged. LCSC stocks both at a few cents; the Harwin header was out
of stock and the pair cost ten dollars a column.

Co-Authored-By: Claude Fable 5.1 <noreply@anthropic.com>
Parts:
- J_LEFT1, J_LEFT2, J_LEFT3: value M20-7910342R -> HX PM2.54-1x3P WT; Ideal Part Number M20-7910342R -> HX PM2.54-1x3P WT; LCSC Part # C3321821 -> C46061767; Order Link https://jlcpcb.com/partdetail/Harwin-M207910342R/C3321821 -> https://www.lcsc.com/product-detail/C46061767.html
- J_RIGHT1, J_RIGHT2, J_RIGHT3: value M20-8890345R -> HX PZ2.54-1x3P WT; Ideal Part Number M20-8890345R -> HX PZ2.54-1x3P WT; LCSC Part # (none) -> C46061676; Order Link https://www.digikey.com/en/products/detail/harwin-inc/M20-8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 -> https://www.lcsc.com/product-detail/C46061676.html; Vendor DigiKey -> LCSC
Changed lines of the file:
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@@
 			)
 		)
-		(property "Value" "M20-7910342R"
+		(property "Value" "HX PM2.54-1x3P WT"
 			(at 45.72 86.36 0)
 			(hide yes)
@@
 			)
 		)
-		(property "Ideal Part Number" "M20-7910342R"
+		(property "Ideal Part Number" "HX PM2.54-1x3P WT"
 			(at 48.26 85.09 0)
 			(hide yes)
@@
 			)
 		)
-		(property "Order Link" "https://jlcpcb.com/partdetail/Harwin-M207910342R/C3321821"
+		(property "Order Link" "https://www.lcsc.com/product-detail/C46061767.html"
 			(at 48.26 85.09 0)
 			(hide yes)
@@
 			)
 		)
-		(property "LCSC Part #" "C3321821"
+		(property "LCSC Part #" "C46061767"
 			(at 48.26 85.09 0)
 			(hide yes)
@@
 			)
 		)
-		(property "Value" "M20-8890345R"
+		(property "Value" "HX PZ2.54-1x3P WT"
 			(at 152.4 93.98 0)
 			(hide yes)
@@
 			)
 		)
-		(property "Ideal Part Number" "M20-8890345R"
+		(property "Ideal Part Number" "HX PZ2.54-1x3P WT"
 			(at 149.86 92.71 0)
 			(hide yes)
@@
 			)
 		)
-		(property "Order Link" "https://www.digikey.com/en/products/detail/harwin-inc/M20-8890345R/6565723"
+		(property "Order Link" "https://www.lcsc.com/product-detail/C46061676.html"
 			(at 149.86 92.71 0)
 			(hide yes)
@@
 			)
 		)
-		(property "Vendor" "DigiKey"
+		(property "Vendor" "LCSC"
 			(at 149.86 92.71 0)
 			(hide yes)
@@
 			)
 		)
-		(property "LCSC Part #" ""
+		(property "LCSC Part #" "C46061676"
 			(at 149.86 92.71 0)
 			(hide yes)
@@
 			)
 		)
-		(property "Value" "M20-8890345R"
+		(property "Value" "HX PZ2.54-1x3P WT"
 			(at 152.4 86.36 0)
 			(hide yes)
@@
 			)
 		)
-		(property "Ideal Part Number" "M20-8890345R"
+		(property "Ideal Part Number" "HX PZ2.54-1x3P WT"
 			(at 149.86 85.09 0)
 			(hide yes)
@@
 			)
 		)
-		(property "Order Link" "https://www.digikey.com/en/products/detail/harwin-inc/M20-8890345R/6565723"
+		(property "Order Link" "https://www.lcsc.com/product-detail/C46061676.html"
 			(at 149.86 85.09 0)
 			(hide yes)
@@
 			)
 		)
-		(property "Vendor" "DigiKey"
+		(property "Vendor" "LCSC"
 			(at 149.86 85.09 0)
 			(hide yes)
@@
 			)
 		)
-		(property "LCSC Part #" ""
+		(property "LCSC Part #" "C46061676"
 			(at 149.86 85.09 0)
 			(hide yes)
@@
 			)
 		)
-		(property "Value" "M20-8890345R"
+		(property "Value" "HX PZ2.54-1x3P WT"
 			(at 152.4 78.74 0)
 			(hide yes)
@@
 			)
 		)
-		(property "Ideal Part Number" "M20-8890345R"
+		(property "Ideal Part Number" "HX PZ2.54-1x3P WT"
 			(at 149.86 77.47 0)
 			(hide yes)
@@
 			)
 		)
-		(property "Order Link" "https://www.digikey.com/en/products/detail/harwin-inc/M20-8890345R/6565723"
+		(property "Order Link" "https://www.lcsc.com/product-detail/C46061676.html"
 			(at 149.86 77.47 0)
 			(hide yes)
@@
 			)
 		)
-		(property "Vendor" "DigiKey"
+		(property "Vendor" "LCSC"
 			(at 149.86 77.47 0)
 			(hide yes)
@@
 			)
 		)
-		(property "LCSC Part #" ""
+		(property "LCSC Part #" "C46061676"
 			(at 149.86 77.47 0)
 			(hide yes)
@@
 			)
 		)
-		(property "Value" "M20-7910342R"
+		(property "Value" "HX PM2.54-1x3P WT"
 			(at 45.72 78.74 0)
 			(hide yes)
@@
 			)
 		)
-		(property "Ideal Part Number" "M20-7910342R"
+		(property "Ideal Part Number" "HX PM2.54-1x3P WT"
 			(at 48.26 77.47 0)
 			(hide yes)
@@
 			)
 		)
-		(property "Order Link" "https://jlcpcb.com/partdetail/Harwin-M207910342R/C3321821"
+		(property "Order Link" "https://www.lcsc.com/product-detail/C46061767.html"
 			(at 48.26 77.47 0)
 			(hide yes)
@@
 			)
 		)
-		(property "LCSC Part #" "C3321821"
+		(property "LCSC Part #" "C46061767"
 			(at 48.26 77.47 0)
 			(hide yes)
@@
 			)
 		)
-		(property "Value" "M20-7910342R"
+		(property "Value" "HX PM2.54-1x3P WT"
 			(at 45.72 93.98 0)
 			(hide yes)
@@
 			)
 		)
-		(property "Ideal Part Number" "M20-7910342R"
+		(property "Ideal Part Number" "HX PM2.54-1x3P WT"
 			(at 48.26 92.71 0)
 			(hide yes)
@@
 			)
 		)
-		(property "Order Link" "https://jlcpcb.com/partdetail/Harwin-M207910342R/C3321821"
+		(property "Order Link" "https://www.lcsc.com/product-detail/C46061767.html"
 			(at 48.26 92.71 0)
 			(hide yes)
@@
 			)
 		)
-		(property "LCSC Part #" "C3321821"
+		(property "LCSC Part #" "C46061767"
 			(at 48.26 92.71 0)
 			(hide yes)

Commit message: Rev 2 key module: switch footprint in the right handedness, rerouted
Own Choc v1 hotswap footprint from the Kailh drawing, socket above each
key, board 16.85 mm wide, connector rows and U1 moved into the new gaps,
fully rerouted. DRC, ERC and schematic parity clean. Fab files and BOM
regenerated; plan doc records where the layout deviates from the plan.

Co-Authored-By: Claude Fable 5.1 <noreply@anthropic.com>
Parts:
- SW1, SW2, SW3, SW4, SW5: footprint kbd:keyswitch_choc12_hotswap_1u -> Library:Kailh_choc_v1_hotswap
Changed lines of the file:
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@@
 			)
 		)
-		(property "Footprint" "kbd:keyswitch_choc12_hotswap_1u"
+		(property "Footprint" "Library:Kailh_choc_v1_hotswap"
 			(at 78.74 104.14 0)
 			(hide yes)
@@
 			)
 		)
-		(property "Footprint" "kbd:keyswitch_choc12_hotswap_1u"
+		(property "Footprint" "Library:Kailh_choc_v1_hotswap"
 			(at 78.74 76.2 0)
 			(hide yes)
@@
 			)
 		)
-		(property "Footprint" "kbd:keyswitch_choc12_hotswap_1u"
+		(property "Footprint" "Library:Kailh_choc_v1_hotswap"
 			(at 78.74 90.17 0)
 			(hide yes)
@@
 			)
 		)
-		(property "Footprint" "kbd:keyswitch_choc12_hotswap_1u"
+		(property "Footprint" "Library:Kailh_choc_v1_hotswap"
 			(at 78.74 119.38 0)
 			(hide yes)
@@
 			)
 		)
-		(property "Footprint" "kbd:keyswitch_choc12_hotswap_1u"
+		(property "Footprint" "Library:Kailh_choc_v1_hotswap"
 			(at 78.74 62.23 0)
 			(hide yes)

Commit message: Fab files carry a revision: v4
Title block, back silkscreen and file names all say v4; Electronics.md
keeps the revision table.

Co-Authored-By: Claude Fable 5.1 <noreply@anthropic.com>
Other:
- company: (none) -> nevyn.dev
- title: (none) -> roamyboard key module
Changed lines of the file:
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@@
 	(generator_version "10.0")
 	(paper "A4")
+	(title_block
+		(title "roamyboard key module")
+		(rev "v4")
+		(company "nevyn.dev")
+	)
 	(junction
 		(at 101.6 82.55)
