File: electronics/KeyModule/KeyModule.kicad_pcb (KiCad board)
At the start: 2 copper layers, 20 x 100 mm, 13 parts, among them SW1 SW_Push, SW2 SW_Push, SW3 SW_Push, SW4 SW_Push, SW5 SW_Push, U1 74HC165

Commit message: just some uncommitted changes :S
Parts:
- removed J_LEFT1: Conn_01x09, Connector_PinHeader_2.54mm:PinHeader_1x09_P2.54mm_Vertical_SMD_Pin1Right
- removed J_RIGHT1: Conn_01x09, Connector_PinHeader_2.54mm:PinHeader_1x09_P2.54mm_Vertical_SMD_Pin1Left
- added REF**: CONN_SMD2, Library:CONN_SMD2, B.Cu at (82.2, 59.4)
- added REF**: CONN_SMD2, Library:CONN_SMD2, B.Cu at (81.4, 116.5)
- added REF**: CONN_SMD2, Library:CONN_SMD2, B.Cu at (82.3, 61.9)
- added REF**: CONN_SMD2, Library:CONN_SMD2, B.Cu at (73.9, 78.7)
- added REF**: CONN_SMD2, Library:CONN_SMD2, B.Cu at (81.4, 119.1)
- added REF**: CONN_SMD2, Library:CONN_SMD2, B.Cu at (82.4, 81.1)
- added REF**: CONN_SMD2, Library:CONN_SMD2, B.Cu at (82.3, 78.6)
- added REF**: CONN_SMD2, Library:CONN_SMD2, B.Cu at (74.1, 59.5)
- added REF**: CONN_SMD2, Library:CONN_SMD2, B.Cu at (74.1, 62.1)
- added REF**: CONN_SMD2, Library:CONN_SMD2, B.Cu at (73.9, 81.2)
- added REF**: CONN_SMD2, Library:CONN_SMD2, B.Cu at (73.7, 118.9)
- added REF**: CONN_SMD2, Library:CONN_SMD2, B.Cu at (73.7, 116.4)
Routing:
- net +5V: track 17.5 -> 0.00 mm
- net +3.3V: track 101.4 -> 118.9 mm
- net Net-(U1-D3): track 44.8 -> 30.8 mm, vias 3 -> 2
- net GND: track 125.3 -> 139.3 mm, vias 2 -> 3
