File: electronics/KeyModule/KeyModule.kicad_pcb (KiCad board)
At the start: 2 copper layers, 16.5 x 100 mm, 17 parts, among them SW1 SW_Push, SW2 SW_Push, SW3 SW_Push, SW4 SW_Push, SW5 SW_Push, U1 74HC165

Commit message: 3d models and shi
Routing:
- net GND: track 139.3 -> 0.00 mm, vias 3 -> 0
- net +3.3V: track 118.9 -> 0.00 mm, vias 2 -> 0
- net Net-(U1-D4): track 54.4 -> 0.00 mm, vias 2 -> 0
- net /PL: track 48.3 -> 0.00 mm, vias 2 -> 0
- net /DATA_IN: track 41.6 -> 0.00 mm, vias 2 -> 0
- net /CLK: track 40.0 -> 0.00 mm, vias 2 -> 0
- net Net-(U1-D0): track 37.0 -> 0.00 mm, vias 1 -> 0
- net Net-(U1-D3): track 30.8 -> 0.00 mm, vias 2 -> 0
- net Net-(U1-D2): track 26.8 -> 0.00 mm, vias 1 -> 0
- net /DATA_OUT: track 23.2 -> 0.00 mm, vias 4 -> 0
- net Net-(U1-D1): track 21.4 -> 0.00 mm, vias 1 -> 0
- net /LED: track 18.0 -> 0.00 mm
- net /SCL: track 17.0 -> 0.00 mm
- net /SDA: track 11.2 -> 0.00 mm
